Commit message: Make gripper close position to be more similar to diameter of coke can
Signed-off-by: Aaron Chong <aaronchongth@gmail.com>

File: panda_moveit_config/srdf/panda_gripper.xacro (robot description, xacro)
@@ -20,6 +20,6 @@
     </group_state>
     <group_state name="close" group="gripper">
-      <joint name="${prefix}finger_joint1" value="0.001"/>
-      <joint name="${prefix}finger_joint2" value="0.001"/>
+      <joint name="${prefix}finger_joint1" value="0.02"/>
+      <joint name="${prefix}finger_joint2" value="0.02"/>
     </group_state>
     <disable_collisions link1="${prefix}hand" link2="${prefix}leftfinger" reason="Adjacent"/>
