Commit message: Add grasp / pregrasp pose, spawn coordinates, detachable joint
Signed-off-by: Luca Della Vedova <lucadv@intrinsic.ai>

File: panda_moveit_config/srdf/panda_arm.xacro (robot description, xacro)
@@ -38,4 +38,22 @@
       <joint name="${prefix}joint7" value="${pi/4}"/>
     </group_state>
+    <group_state group="arm" name="pre_grasp">
+      <joint name="${prefix}joint1" value="-0.192"/>
+      <joint name="${prefix}joint2" value="0.297"/>
+      <joint name="${prefix}joint3" value="0"/>
+      <joint name="${prefix}joint4" value="-1.99"/>
+      <joint name="${prefix}joint5" value="0"/>
+      <joint name="${prefix}joint6" value="2.27"/>
+      <joint name="${prefix}joint7" value="0"/>
+    </group_state>
+    <group_state group="arm" name="grasp">
+      <joint name="${prefix}joint1" value="-0.192"/>
+      <joint name="${prefix}joint2" value="0.47"/>
+      <joint name="${prefix}joint3" value="0"/>
+      <joint name="${prefix}joint4" value="-2.02"/>
+      <joint name="${prefix}joint5" value="0"/>
+      <joint name="${prefix}joint6" value="2.48"/>
+      <joint name="${prefix}joint7" value="0"/>
+    </group_state>
     <disable_collisions link1="${prefix}link0" link2="${prefix}link1" reason="Adjacent"/>
     <disable_collisions link1="${prefix}link0" link2="${prefix}link2" reason="Never"/>

Commit message: Add drop poses
Signed-off-by: Luca Della Vedova <lucadv@intrinsic.ai>

File: panda_moveit_config/srdf/panda_arm.xacro (robot description, xacro)
@@ -56,4 +56,22 @@
       <joint name="${prefix}joint7" value="0"/>
     </group_state>
+    <group_state group="arm" name="pre_drop">
+      <joint name="${prefix}joint1" value="0.73"/>
+      <joint name="${prefix}joint2" value="0.63"/>
+      <joint name="${prefix}joint3" value="0.70"/>
+      <joint name="${prefix}joint4" value="-2.01"/>
+      <joint name="${prefix}joint5" value="-0.59"/>
+      <joint name="${prefix}joint6" value="-2.41"/>
+      <joint name="${prefix}joint7" value="0"/>
+    </group_state>
+    <group_state group="arm" name="drop">
+      <joint name="${prefix}joint1" value="1.03"/>
+      <joint name="${prefix}joint2" value="1.26"/>
+      <joint name="${prefix}joint3" value="0.35"/>
+      <joint name="${prefix}joint4" value="-1.61"/>
+      <joint name="${prefix}joint5" value="-0.87"/>
+      <joint name="${prefix}joint6" value="2.70"/>
+      <joint name="${prefix}joint7" value="0"/>
+    </group_state>
     <disable_collisions link1="${prefix}link0" link2="${prefix}link1" reason="Adjacent"/>
     <disable_collisions link1="${prefix}link0" link2="${prefix}link2" reason="Never"/>

Commit message: Tune limits and predrop pose
Signed-off-by: Luca Della Vedova <lucadellavr@gmail.com>

File: panda_moveit_config/srdf/panda_arm.xacro (robot description, xacro)
@@ -49,18 +49,18 @@
     <group_state group="arm" name="grasp">
       <joint name="${prefix}joint1" value="-0.192"/>
-      <joint name="${prefix}joint2" value="0.47"/>
+      <joint name="${prefix}joint2" value="0.52"/>
       <joint name="${prefix}joint3" value="0"/>
       <joint name="${prefix}joint4" value="-2.02"/>
       <joint name="${prefix}joint5" value="0"/>
-      <joint name="${prefix}joint6" value="2.48"/>
+      <joint name="${prefix}joint6" value="2.53"/>
       <joint name="${prefix}joint7" value="0"/>
     </group_state>
     <group_state group="arm" name="pre_drop">
-      <joint name="${prefix}joint1" value="0.73"/>
-      <joint name="${prefix}joint2" value="0.63"/>
-      <joint name="${prefix}joint3" value="0.70"/>
-      <joint name="${prefix}joint4" value="-2.01"/>
-      <joint name="${prefix}joint5" value="-0.59"/>
-      <joint name="${prefix}joint6" value="-2.41"/>
+      <joint name="${prefix}joint1" value="0.98"/>
+      <joint name="${prefix}joint2" value="1.06"/>
+      <joint name="${prefix}joint3" value="0.42"/>
+      <joint name="${prefix}joint4" value="-1.78"/>
+      <joint name="${prefix}joint5" value="-0.84"/>
+      <joint name="${prefix}joint6" value="2.65"/>
       <joint name="${prefix}joint7" value="0"/>
     </group_state>

File: panda_moveit_config/srdf/panda_gripper.xacro (robot description, xacro)
@@ -16,10 +16,10 @@
     </group>
     <group_state name="open" group="gripper">
-      <joint name="${prefix}finger_joint1" value="0.04"/>
-      <joint name="${prefix}finger_joint2" value="0.04"/>
+      <joint name="${prefix}finger_joint1" value="0.039"/>
+      <joint name="${prefix}finger_joint2" value="0.039"/>
     </group_state>
     <group_state name="close" group="gripper">
-      <joint name="${prefix}finger_joint1" value="0.0"/>
-      <joint name="${prefix}finger_joint2" value="0.0"/>
+      <joint name="${prefix}finger_joint1" value="0.001"/>
+      <joint name="${prefix}finger_joint2" value="0.001"/>
     </group_state>
     <disable_collisions link1="${prefix}hand" link2="${prefix}leftfinger" reason="Adjacent"/>

Commit message: Update poses
Signed-off-by: Xiyu Oh <xiyu@openrobotics.org>

File: panda_moveit_config/srdf/panda_arm.xacro (robot description, xacro)
@@ -39,38 +39,38 @@
     </group_state>
     <group_state group="arm" name="pre_grasp">
-      <joint name="${prefix}joint1" value="-0.192"/>
-      <joint name="${prefix}joint2" value="0.297"/>
-      <joint name="${prefix}joint3" value="0"/>
-      <joint name="${prefix}joint4" value="-1.99"/>
-      <joint name="${prefix}joint5" value="0"/>
-      <joint name="${prefix}joint6" value="2.27"/>
-      <joint name="${prefix}joint7" value="0"/>
+      <joint name="${prefix}joint1" value="0.0174533"/>
+      <joint name="${prefix}joint2" value="0.296706"/>
+      <joint name="${prefix}joint3" value="0.10472"/>
+      <joint name="${prefix}joint4" value="-1.93732"/>
+      <joint name="${prefix}joint5" value="-0.0349066"/>
+      <joint name="${prefix}joint6" value="2.21657"/>
+      <joint name="${prefix}joint7" value="0.331613"/>
     </group_state>
     <group_state group="arm" name="grasp">
-      <joint name="${prefix}joint1" value="-0.192"/>
-      <joint name="${prefix}joint2" value="0.52"/>
-      <joint name="${prefix}joint3" value="0"/>
-      <joint name="${prefix}joint4" value="-2.02"/>
-      <joint name="${prefix}joint5" value="0"/>
-      <joint name="${prefix}joint6" value="2.53"/>
-      <joint name="${prefix}joint7" value="0"/>
+      <joint name="${prefix}joint1" value="0.0349066"/>
+      <joint name="${prefix}joint2" value="0.541052"/>
+      <joint name="${prefix}joint3" value="0.0872665"/>
+      <joint name="${prefix}joint4" value="-1.98968"/>
+      <joint name="${prefix}joint5" value="-0.0698132"/>
+      <joint name="${prefix}joint6" value="2.49582"/>
+      <joint name="${prefix}joint7" value="0.349066"/>
     </group_state>
     <group_state group="arm" name="pre_drop">
-      <joint name="${prefix}joint1" value="0.98"/>
-      <joint name="${prefix}joint2" value="1.06"/>
-      <joint name="${prefix}joint3" value="0.42"/>
-      <joint name="${prefix}joint4" value="-1.78"/>
-      <joint name="${prefix}joint5" value="-0.84"/>
-      <joint name="${prefix}joint6" value="2.65"/>
-      <joint name="${prefix}joint7" value="0"/>
+      <joint name="${prefix}joint1" value="1.50098"/>
+      <joint name="${prefix}joint2" value="1.37881"/>
+      <joint name="${prefix}joint3" value="0.558505"/>
+      <joint name="${prefix}joint4" value="-0.959931"/>
+      <joint name="${prefix}joint5" value="-0.663225"/>
+      <joint name="${prefix}joint6" value="2.16421"/>
+      <joint name="${prefix}joint7" value="0.0523599"/>
     </group_state>
     <group_state group="arm" name="drop">
-      <joint name="${prefix}joint1" value="1.03"/>
-      <joint name="${prefix}joint2" value="1.26"/>
-      <joint name="${prefix}joint3" value="0.35"/>
-      <joint name="${prefix}joint4" value="-1.61"/>
-      <joint name="${prefix}joint5" value="-0.87"/>
-      <joint name="${prefix}joint6" value="2.70"/>
-      <joint name="${prefix}joint7" value="0"/>
+      <joint name="${prefix}joint1" value="1.72788"/>
+      <joint name="${prefix}joint2" value="1.5708"/>
+      <joint name="${prefix}joint3" value="0.15708"/>
+      <joint name="${prefix}joint4" value="-0.645772"/>
+      <joint name="${prefix}joint5" value="-0.174533"/>
+      <joint name="${prefix}joint6" value="2.19911"/>
+      <joint name="${prefix}joint7" value="-0.122173"/>
     </group_state>
     <disable_collisions link1="${prefix}link0" link2="${prefix}link1" reason="Adjacent"/>

Commit message: Joint7 set to 0
Signed-off-by: Xiyu Oh <xiyu@openrobotics.org>

File: panda_moveit_config/srdf/panda_arm.xacro (robot description, xacro)
@@ -45,5 +45,5 @@
       <joint name="${prefix}joint5" value="-0.0349066"/>
       <joint name="${prefix}joint6" value="2.21657"/>
-      <joint name="${prefix}joint7" value="0.331613"/>
+      <joint name="${prefix}joint7" value="0"/>
     </group_state>
     <group_state group="arm" name="grasp">
@@ -54,5 +54,5 @@
       <joint name="${prefix}joint5" value="-0.0698132"/>
       <joint name="${prefix}joint6" value="2.49582"/>
-      <joint name="${prefix}joint7" value="0.349066"/>
+      <joint name="${prefix}joint7" value="0"/>
     </group_state>
     <group_state group="arm" name="pre_drop">
@@ -63,5 +63,5 @@
       <joint name="${prefix}joint5" value="-0.663225"/>
       <joint name="${prefix}joint6" value="2.16421"/>
-      <joint name="${prefix}joint7" value="0.0523599"/>
+      <joint name="${prefix}joint7" value="0"/>
     </group_state>
     <group_state group="arm" name="drop">
@@ -72,5 +72,5 @@
       <joint name="${prefix}joint5" value="-0.174533"/>
       <joint name="${prefix}joint6" value="2.19911"/>
-      <joint name="${prefix}joint7" value="-0.122173"/>
+      <joint name="${prefix}joint7" value="0"/>
     </group_state>
     <disable_collisions link1="${prefix}link0" link2="${prefix}link1" reason="Adjacent"/>

Commit message: Joint values for office world
Signed-off-by: Xiyu Oh <xiyu@openrobotics.org>

File: panda_moveit_config/srdf/panda_arm.xacro (robot description, xacro)
@@ -12,11 +12,11 @@
     </group>
     <group_state group="arm" name="ready">
-      <joint name="${prefix}joint1" value="0"/>
-      <joint name="${prefix}joint2" value="${-pi/4}"/>
-      <joint name="${prefix}joint3" value="0"/>
-      <joint name="${prefix}joint4" value="${-135*pi/180}"/>
-      <joint name="${prefix}joint5" value="0"/>
-      <joint name="${prefix}joint6" value="${pi/2}"/>
-      <joint name="${prefix}joint7" value="${pi/4}"/>
+      <joint name="${prefix}joint1" value="1.39626"/>
+      <joint name="${prefix}joint2" value="-0.244346"/>
+      <joint name="${prefix}joint3" value="-2.23402"/>
+      <joint name="${prefix}joint4" value="-1.20428"/>
+      <joint name="${prefix}joint5" value="-0.20944"/>
+      <joint name="${prefix}joint6" value="1.3439"/>
+      <joint name="${prefix}joint7" value="0"/>
     </group_state>
     <group_state group="arm" name="extended">
@@ -39,37 +39,37 @@
     </group_state>
     <group_state group="arm" name="pre_grasp">
-      <joint name="${prefix}joint1" value="-0.192"/>
-      <joint name="${prefix}joint2" value="0.297"/>
-      <joint name="${prefix}joint3" value="0"/>
-      <joint name="${prefix}joint4" value="-1.99"/>
-      <joint name="${prefix}joint5" value="0"/>
-      <joint name="${prefix}joint6" value="2.27"/>
+      <joint name="${prefix}joint1" value="-0.10472"/>
+      <joint name="${prefix}joint2" value="-0.174533"/>
+      <joint name="${prefix}joint3" value="-1.46608"/>
+      <joint name="${prefix}joint4" value="-2.3911"/>
+      <joint name="${prefix}joint5" value="-0.15708"/>
+      <joint name="${prefix}joint6" value="2.3911"/>
       <joint name="${prefix}joint7" value="0"/>
     </group_state>
     <group_state group="arm" name="grasp">
-      <joint name="${prefix}joint1" value="-0.192"/>
-      <joint name="${prefix}joint2" value="0.52"/>
-      <joint name="${prefix}joint3" value="0"/>
-      <joint name="${prefix}joint4" value="-2.02"/>
-      <joint name="${prefix}joint5" value="0"/>
-      <joint name="${prefix}joint6" value="2.53"/>
+      <joint name="${prefix}joint1" value="0.488692"/>
+      <joint name="${prefix}joint2" value="-0.383972"/>
+      <joint name="${prefix}joint3" value="-2.11185"/>
+      <joint name="${prefix}joint4" value="-2.3911"/>
+      <joint name="${prefix}joint5" value="-0.488692"/>
+      <joint name="${prefix}joint6" value="2.56563"/>
       <joint name="${prefix}joint7" value="0"/>
     </group_state>
     <group_state group="arm" name="pre_drop">
-      <joint name="${prefix}joint1" value="0.98"/>
-      <joint name="${prefix}joint2" value="1.06"/>
-      <joint name="${prefix}joint3" value="0.42"/>
-      <joint name="${prefix}joint4" value="-1.78"/>
-      <joint name="${prefix}joint5" value="-0.84"/>
-      <joint name="${prefix}joint6" value="2.65"/>
+      <joint name="${prefix}joint1" value="2.02458"/>
+      <joint name="${prefix}joint2" value="-0.872665"/>
+      <joint name="${prefix}joint3" value="-2.53073"/>
+      <joint name="${prefix}joint4" value="-1.76278"/>
+      <joint name="${prefix}joint5" value="-0.715585"/>
+      <joint name="${prefix}joint6" value="2.40855"/>
       <joint name="${prefix}joint7" value="0"/>
     </group_state>
     <group_state group="arm" name="drop">
-      <joint name="${prefix}joint1" value="1.03"/>
-      <joint name="${prefix}joint2" value="1.26"/>
-      <joint name="${prefix}joint3" value="0.35"/>
-      <joint name="${prefix}joint4" value="-1.61"/>
-      <joint name="${prefix}joint5" value="-0.87"/>
-      <joint name="${prefix}joint6" value="2.70"/>
+      <joint name="${prefix}joint1" value="2.25147"/>
+      <joint name="${prefix}joint2" value="-1.6057"/>
+      <joint name="${prefix}joint3" value="-2.74017"/>
+      <joint name="${prefix}joint4" value="-1.11701"/>
+      <joint name="${prefix}joint5" value="-0.820305"/>
+      <joint name="${prefix}joint6" value="2.58309"/>
       <joint name="${prefix}joint7" value="0"/>
     </group_state>
